File: dropout-miniusb/dropout-miniusb.sch (KiCad schematic (older format))
At the start: 45 parts, among them SW1 Rotary_Encoder_Switch, SW2 SW_Push, U1 ProMicro

Commit message: micro usb promicro
Parts:
- R1: value 680 -> 330
- U1: footprint promicro:ProMicro -> promicro:ProMicro_MiniUsb
Changed lines of the file:
@@
 P 3400 1800
 F 0 "R1" H 3330 1754 50  0000 R CNN
-F 1 "680" H 3330 1845 50  0000 R CNN
+F 1 "330" H 3330 1845 50  0000 R CNN
 F 2 "Resistor_SMD:R_0805_2012Metric_Pad1.15x1.40mm_HandSolder" V 3330 1800 50  0001 C CNN
 F 3 "~" H 3400 1800 50  0001 C CNN
@@
 F 0 "U1" H 7650 5737 60  0000 C CNN
 F 1 "ProMicro" H 7650 5631 60  0000 C CNN
-F 2 "promicro:ProMicro" H 7750 3650 60  0001 C CNN
+F 2 "promicro:ProMicro_MiniUsb" H 7750 3650 60  0001 C CNN
 F 3 "" H 7750 3650 60  0000 C CNN
 	1    7650 4700

Commit message: firmware
Parts:
- added C1, C2: 10nF, Capacitor_SMD:C_0805_2012Metric_Pad1.15x1.40mm_HandSolder, symbol Device:C
Connections:
- wire segments 115 -> 119
Changed lines of the file:
@@
 	6850 4150 6950 4150
 Wire Wire Line
-	6350 2300 6600 2300
-Wire Wire Line
-	6350 2100 6600 2100
+	6350 2100 6550 2100
 Wire Wire Line
 	6350 2200 7000 2200
@@
 Wire Wire Line
 	9800 5050 9800 5250
+$Comp
+L Device:C C2
+U 1 1 5FCA2C97
+P 6550 2450
+F 0 "C2" H 6665 2496 50  0000 L CNN
+F 1 "10nF" H 6665 2405 50  0000 L CNN
+F 2 "Capacitor_SMD:C_0805_2012Metric_Pad1.15x1.40mm_HandSolder" H 6588 2300 50  0001 C CNN
+F 3 "~" H 6550 2450 50  0001 C CNN
+	1    6550 2450
+	1    0    0    -1
+$EndComp
+$Comp
+L Device:C C1
+U 1 1 5FCA364C
+P 6550 1950
+F 0 "C1" H 6665 1996 50  0000 L CNN
+F 1 "10nF" H 6665 1905 50  0000 L CNN
+F 2 "Capacitor_SMD:C_0805_2012Metric_Pad1.15x1.40mm_HandSolder" H 6588 1800 50  0001 C CNN
+F 3 "~" H 6550 1950 50  0001 C CNN
+	1    6550 1950
+	1    0    0    -1
+$EndComp
+Connection ~ 6550 2100
+Wire Wire Line
+	6550 2100 6600 2100
+Connection ~ 6550 2300
+Wire Wire Line
+	6550 2300 6600 2300
+Wire Wire Line
+	6350 2300 6550 2300
+$Comp
+L power:GND #PWR0102
+U 1 1 5FCA3F65
+P 6550 2750
+F 0 "#PWR0102" H 6550 2500 50  0001 C CNN
+F 1 "GND" H 6555 2577 50  0000 C CNN
+F 2 "" H 6550 2750 50  0001 C CNN
+F 3 "" H 6550 2750 50  0001 C CNN
+	1    6550 2750
+	1    0    0    -1
+$EndComp
+$Comp
+L power:GND #PWR0103
+U 1 1 5FCA4369
+P 7100 1800
+F 0 "#PWR0103" H 7100 1550 50  0001 C CNN
+F 1 "GND" H 7105 1627 50  0000 C CNN
+F 2 "" H 7100 1800 50  0001 C CNN
+F 3 "" H 7100 1800 50  0001 C CNN
+	1    7100 1800
+	1    0    0    -1
+$EndComp
+Wire Wire Line
+	6550 2600 6550 2750
+Wire Wire Line
+	6550 1800 7100 1800
 $EndSCHEMATC
